File: MainBoard.sch (EAGLE design)
At the start: 0 parts

Commit message: Schematic for audio section
Parts:
- added C1, C10, C11, C2, C3, C4, C6, C7, C8, C9: 1µF, microbuilder:CAP_CERAMIC0805-NOOUTLINE
- added C5: 2.2u, microbuilder:CAP_CERAMIC0805-NOOUTLINE
- added J1: 22-27-2101-10, con-molex:22-27-2101-10
- added R1, R2: 10K, microbuilder:RESISTOR0805_NOOUTLINE
- added R3, R4, R5, R6: 100K, microbuilder:RESISTOR0805_NOOUTLINE
- added U1: microSD, SparkFun:USD-SOCKETSMD
- added U2: TPA2016, tpa2016:TPA2016
- added U3: AK4430ET, AK4430ET:AK4430ET
- added X1, X2, X3: 22-23-2021, con-molex:22-23-2021
Connections:
- new net +3V3: C10.2, C11.1, C3.2, C8.2, R1.1, R2.2, R3.2, R6.1, U1.NC, U2.AVDD, U3.CVDD, U3.VDD
- new net AGND: C10.1, C4.1, C5.1, R4.1, R5.1, U2.AGND, U2.INL-, U2.INR-, U3.VSS1
- new net GND: C11.2, C3.1, U1.CD2, U1.GND, U1.SHIELD1, U1.SHIELD2, U2.PGND
- new net I2SBICK: U3.BICK
- new net I2SLRCK: U3.LRCK
- new net I2SMCLK: U3.MCLK
- new net I2SSDTI: U3.SDTI
- new net MMCCD: R6.2, U1.CD1
- new net MMCCS: U1.CS
- new net MMCDI: U1.DI
- new net MMCSCK: U1.SCK
- new net MMCSDO: U1.DO
- new net MUTE: R1.2, R5.2, U2.SDZ, U3.SMUTE
- new net N$1: U2.OUTL+, X1-1.S
- new net N$10: C8.1, C9.1, U3.VSS2
- new net N$12: C9.2, U3.VEE
- new net N$13: C6.1, U3.CN
- new net N$14: C6.2, U3.CP
- new net N$15: R4.2, U3.DIF
- new net N$2: U2.OUTL-, X1-2.S
- new net N$3: U2.OUTR+, X2-1.S
- new net N$4: C2.1, U3.AOUTR
- new net N$5: C1.1, U3.AOUTL
- new net N$6: C1.2, U2.INL+
- new net N$7: C2.2, U2.INR+
- new net N$8: U2.OUTR-, X2-2.S
- new net N$9: C5.2, U3.VREFH
- new net SCL: R2.1, U2.SCL
- new net SDA: R3.1, U2.SDA
- new net V+: C4.2, U2.PVDDL, U2.PVDDR
- new net VCC: U1.VCC
