File: MainBoard.sch (EAGLE design)
At the start: 24 parts, among them J1 22-27-2101-10, U1 microSD, U2 TPA2016, U3 AK4430ET, X1 22-23-2021, X2 22-23-2021, X3 22-23-2021

Commit message: Switched to SMT for power jack and headphones
Parts:
- removed J1: 22-27-2101-10, con-molex:22-27-2101-10
- removed X2, X3: 22-23-2021, con-molex:22-23-2021
- added C12, C13, C14: 2.2u, microbuilder:CAP_CERAMIC0805-NOOUTLINE
- added C15, C16, C17: 1µF, microbuilder:CAP_CERAMIC0805-NOOUTLINE
- added CN1, CN2, CN3: (no value), adafruit:JST_2PIN-SMT-RA
- added D3: (no value), diode:ZENER-DIODESOD80C
- added R7: 100K, microbuilder:RESISTOR0805_NOOUTLINE
- added U$1: 3,5MMPHONO, sj1-351x:3,5MMPHONO
- added U$2: PJ-002AH, PJ-002AH-SMT:PJ-002AH
- added U11: PIC32MX110QFN, pic32mx110:PIC32MX110QFN
- added U12: CSTCE, CSTCE:CSTCE
- X1: value 22-23-2021 -> C-GRID-08-15-91; device con-molex:22-23-2021 -> con-molex:C-GRID-08-15-91
Connections:
- new net !MCLR: R7.1, U11.!MCLR
- new net N$11: C13.2, U11.VCAP
- new net N$16: U11.AN9/C3INA/RPB15/SCK2/CTED6/PMCS1/RB15
- new net N$17: U11.CVREFOUT/AN10/C3INB/RPB14/SCK1/CTED5/PMWR/RB14
- new net N$18: U11.AN11/RPB13/CTPLS/PMRD/RB13
- new net N$19: U11.PGEC2/TMS/RPB11/PMD1/RB11
- new net N$20: U11.PGED2/RPB10/CTED11/PMD2/RB10
- new net N$21: U11.TDO/RPB9/SDA1/CTED4/PMD3/RB9
- new net N$22: U11.TCK/RPB8/SCL1/CTED10/PMD4/RB8
- new net N$24: U11.AN5/C1INA/C2INC/RTCC/RPB3/SCL2/RB3
- new net N$25: U11.AN4/C1INB/C2IND/RPB2/SDA2/CTED13/RB2
- new net N$26: U11.PGEC1/AN3/C1INC/C2INA/RPB1/CTED12/RB1
- new net N$27: U11.PGED1/AN2/C1IND/C2INB/C3IND/RPB0/RB0
- new net N$28: U11.SOSCO/RPA4/T1CK/CTED9/PMA1/RA4
- new net N$29: U11.VREF-/CVREF-/AN1/RPA1/CTED2/RA1
- new net N$31: CN1.1, U$2.3
- new net N$33: U$1.2, U3.AOUTL
- new net N$34: U$1.3, U3.AOUTR
- new net N$36: CN1.2, D3.A, U$2.1
- new net PGC: U11.PGEC3/RPB6/PMD6/RB6
- new net PGD: U11.PGED3/RPB5/PMD7/RB5
- new net RIRQ: X1-5.S
- new net RMISO: X1-4.S
- new net RMOSI: X1-3.S
- new net RRST: X1-7.S
- new net RSCK: X1-2.S
- new net RSDA: X1-1.S
- new net XI: U11.OSC1/CLKI/RPA2/RA2, U12.3
- new net XO: U11.OSC2/CLKO/RPA3/PMA0/RA3, U12.1
- net +3V3: now also C12.2, C14.2, R7.2, U11.VSS, U11.VSS2, X1-8.S
- net AGND: now also C15.1, C16.1, C17.1, U$1.1, U$2.2
- net GND: now also C12.1, C13.1, C14.1, U11.AVDD, U11.AVSS, U11.VDD, U12.2, X1-6.S
- net N$1: now also CN2.2; no longer X1-1.S
- net N$2: now also CN2.1; no longer X1-2.S
- net N$3: now also CN3.2; no longer X2-1.S
- net N$4: now also U$1.5; no longer U3.AOUTR
- net N$5: now also U$1.4; no longer U3.AOUTL
- net N$8: now also CN3.1; no longer X2-2.S
- net VCC: now also C15.2, C16.2, C17.2, D3.C
Other:
- note added: "D3 use B130LB-13-F"
- note added: "J1 use EJ508A"
- moved on the sheet: X1-1, X1-2

Commit message: More routing
Parts:
- removed C3, C7, C8: 1µF, microbuilder:CAP_CERAMIC0805-NOOUTLINE
- added C18: 1µF, microbuilder:CAP_CERAMIC0805-NOOUTLINE
- added C21: 10pF, microbuilder:CAP_CERAMIC0603_NO
- added C22, C23, C24: 22uF/10V X5R, microbuilder:CAP_CERAMIC0805-NOOUTLINE
- added C25: 1uF/10V X5R, microbuilder:CAP_CERAMIC0805-NOOUTLINE
- added L1: NRS5030T1R0NMGJ, microbuilder:INDUCTORTDK_VLC5045
- added R12, R13, R9: 105K, microbuilder:RESISTOR_0603_NOOUT
- added R8: 1M, microbuilder:RESISTOR_0603_NOOUT
- added RN1: (no value), resistor-dil:4R-N0402ARV341
- added U$3: JST-4PIN, adafruit:JST-4PIN
- added U4: TPS63060, microbuilder:VREG_TPS63060/1
- added X2: 22-23-2051, con-molex:22-23-2051
- C1, C10, C11, C12, C13, C14, C2, C5, C6, C9: device microbuilder:CAP_CERAMIC0805-NOOUTLINE -> microbuilder:CAP_CERAMIC0603_NO
- R1, R2, R3, R4, R5, R6, R7: device microbuilder:RESISTOR0805_NOOUTLINE -> microbuilder:RESISTOR_0603_NOOUT
Connections:
- net N$33 renamed AOUTL
- net N$34 renamed AOUTR
- removed net MMCDI: U1.DI
- removed net MMCSDO: U1.DO
- removed net N$17: U11.CVREFOUT/AN10/C3INB/RPB14/SCK1/CTED5/PMWR/RB14
- removed net N$19: U11.PGEC2/TMS/RPB11/PMD1/RB11
- removed net N$20: U11.PGED2/RPB10/CTED11/PMD2/RB10
- removed net N$21: U11.TDO/RPB9/SDA1/CTED4/PMD3/RB9
- removed net N$22: U11.TCK/RPB8/SCL1/CTED10/PMD4/RB8
- removed net N$24: U11.AN5/C1INA/C2INC/RTCC/RPB3/SCL2/RB3
- removed net N$25: U11.AN4/C1INB/C2IND/RPB2/SDA2/CTED13/RB2
- removed net N$27: U11.PGED1/AN2/C1IND/C2INB/C3IND/RPB0/RB0
- removed net N$28: U11.SOSCO/RPA4/T1CK/CTED9/PMA1/RA4
- removed net N$29: U11.VREF-/CVREF-/AN1/RPA1/CTED2/RA1
- removed net RMISO: X1-4.S
- removed net RMOSI: X1-3.S
- removed net RSCK: X1-2.S
- removed net RSDA: X1-1.S
- removed net V+: C4.2, U2.PVDDL, U2.PVDDR
- new net ENABLE: R12.2, U4.EN
- new net N$30: L1.2, U4.L2
- new net N$32: U4.VAUX
- new net N$33: C21.1, R8.1, R9.2, U4.FB
- new net PS: R13.1, U4.PSYNC
- new net RFIDSS: U11.PGEC2/TMS/RPB11/PMD1/RB11, X1-1.S
- new net SDI: U1.DO, U11.PGEC1/AN3/C1INC/C2INA/RPB1/CTED12/RB1, X1-4.S
- new net SDO: U1.DI, U11.AN4/C1INB/C2IND/RPB2/SDA2/CTED13/RB2, X1-3.S
- net !MCLR: now also X2-1.S
- net +3V3: now also C18.2, C22.1, C23.1, C24.1, C25.1, C4.2, R8.2, U$3.3, U2.PVDDL, U2.PVDDR, U4.VOUT; no longer C3.2, C8.2
- net AGND: no longer C10.1, C15.1, C16.1, C17.1, C4.1, C5.1, R5.1, U$1.1, U$2.2, U2.AGND, U2.INL-, U2.INR-, U3.VSS1
- net GND: now also C10.1, C15.1, C16.1, C17.1, C18.1, C21.2, C22.2, C23.2, C24.2, C25.2, C4.1, C5.1, C9.1, R13.2, R5.1, R9.1, U$1.1, U$2.2, U$3.4, U2.AGND, U2.INL-, U2.INR-, U3.VSS1, U3.VSS2, U4.GND, U4.PGND, X2-3.S; no longer C3.1
- net I2SBICK: now also RN1C.1, RN1C.2, U11.AN9/C3INA/RPB15/SCK2/CTED6/PMCS1/RB15
- net I2SLRCK: now also RN1A.1, RN1A.2, U11.PGED2/RPB10/CTED11/PMD2/RB10
- net I2SMCLK: now also RN1D.1, RN1D.2, U11.VREF-/CVREF-/AN1/RPA1/CTED2/RA1
- net I2SSDTI: now also RN1B.1, RN1B.2, U11.SOSCO/RPA4/T1CK/CTED9/PMA1/RA4
- net MMCCD: now also U11.PGED1/AN2/C1IND/C2INB/C3IND/RPB0/RB0
- net MMCCS: now also U11.AN5/C1INA/C2INC/RTCC/RPB3/SCL2/RB3
- net MMCSCK: now also U11.CVREFOUT/AN10/C3INB/RPB14/SCK1/CTED5/PMWR/RB14, X1-2.S
- net N$10: now also L1.1, U4.L1; no longer C8.1, C9.1, U3.VSS2
- net N$16: now also U11.AN12/PMD0/RB12; no longer U11.AN9/C3INA/RPB15/SCK2/CTED6/PMCS1/RB15
- net N$26: now also U11.VREF+/CVREF+/AN0/C3INC/RPA0/CTED1/RA0; no longer U11.PGEC1/AN3/C1INC/C2INA/RPB1/CTED12/RB1
- net N$3: now also U2.OUTR-; no longer U2.OUTR+
- net N$8: now also U2.OUTR+; no longer U2.OUTR-
- net PGC: now also X2-5.S
- net PGD: now also X2-4.S
- net RIRQ: now also U11.SOSCI/RPB4/RB4
- net RRST: now also U11.TDI/RPB7/CTED3/PMD5/INT0/RB7
- net SCL: now also U$3.2, U11.TCK/RPB8/SCL1/CTED10/PMD4/RB8
- net SDA: now also U$3.1, U11.TDO/RPB9/SDA1/CTED4/PMD3/RB9
- net VCC: now also R12.1, U4.VIN; no longer U1.VCC
Other:
- moved on the sheet: R4, R5, X1-1, X1-2, X1-3, X1-4, X1-5, X1-6, X1-7, X1-8

Commit message: copper done
Parts:
- removed RN1: (no value), resistor-dil:4R-N0402ARV341
- added R10, R11: 105K, microbuilder:RESISTOR_0603_NOOUT
Connections:
- net N$16 renamed VSENSE
- removed net N$18: U11.AN11/RPB13/CTPLS/PMRD/RB13
- removed net N$26: U11.VREF+/CVREF+/AN0/C3INC/RPA0/CTED1/RA0
- new net BATS: R10.1, R11.2, U11.VREF+/CVREF+/AN0/C3INC/RPA0/CTED1/RA0
- net +3V3: now also U1.VCC; no longer U1.NC
- net GND: now also R11.1
- net I2SBICK: no longer RN1C.1, RN1C.2
- net I2SLRCK: no longer RN1A.1, RN1A.2
- net I2SMCLK: no longer RN1D.1, RN1D.2
- net I2SSDTI: no longer RN1B.1, RN1B.2
- net MUTE: now also U11.AN11/RPB13/CTPLS/PMRD/RB13
- net VCC: now also R10.2
Changed lines of the file:
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@@
 <part name="GND9" library="supply1" deviceset="GND" device=""/>
 <part name="+3V14" library="supply1" deviceset="+3V3" device=""/>
-<part name="RN1" library="resistor-dil" deviceset="4R-N" device="0402ARV341"/>
 <part name="C18" library="microbuilder" deviceset="CAP_CERAMIC" device="0805-NOOUTLINE" value="1µF"/>
 <part name="X2" library="con-molex" deviceset="22-23-2051" device=""/>
@@
 <part name="+3V17" library="supply1" deviceset="+3V3" device=""/>
 <part name="GND16" library="supply1" deviceset="GND" device=""/>
+<part name="+3V18" library="supply1" deviceset="+3V3" device=""/>
+<part name="R10" library="microbuilder" deviceset="RESISTOR" device="_0603_NOOUT" value="105K"/>
+<part name="R11" library="microbuilder" deviceset="RESISTOR" device="_0603_NOOUT" value="105K"/>
+<part name="U$16" library="microbuilder" deviceset="GND" device=""/>
 </parts>
 <sheets>
@@
 <instance part="GND9" gate="1" x="342.9" y="0" rot="R270"/>
 <instance part="+3V14" gate="G$1" x="342.9" y="10.16"/>
-<instance part="RN1" gate="A" x="119.38" y="33.02"/>
-<instance part="RN1" gate="B" x="119.38" y="27.94"/>
-<instance part="RN1" gate="C" x="119.38" y="30.48"/>
-<instance part="RN1" gate="D" x="119.38" y="50.8"/>
 <instance part="C18" gate="G$1" x="287.02" y="17.78" rot="R180"/>
 <instance part="X2" gate="-1" x="396.24" y="-71.12"/>
@@
 <instance part="+3V17" gate="G$1" x="241.3" y="7.62" rot="R90"/>
 <instance part="GND16" gate="1" x="236.22" y="40.64" rot="R270"/>
+<instance part="+3V18" gate="G$1" x="25.4" y="27.94" smashed="yes" rot="R270">
+<attribute name="VALUE" x="27.94" y="27.94" size="1.778" layer="96"/>
+</instance>
+<instance part="R10" gate="G$1" x="71.12" y="-33.02" rot="R90"/>
+<instance part="R11" gate="G$1" x="71.12" y="-45.72" rot="R90"/>
+<instance part="U$16" gate="G$1" x="71.12" y="-53.34"/>
 </instances>
 <busses>
@@
 <junction x="88.9" y="-27.94"/>
 <junction x="81.28" y="-27.94"/>
-<wire x1="81.28" y1="-27.94" x2="66.04" y2="-27.94" width="0.1524" layer="91"/>
+<wire x1="81.28" y1="-27.94" x2="71.12" y2="-27.94" width="0.1524" layer="91"/>
 <pinref part="D3" gate="G$1" pin="C"/>
+<pinref part="R10" gate="G$1" pin="2"/>
+<wire x1="71.12" y1="-27.94" x2="66.04" y2="-27.94" width="0.1524" layer="91"/>
+<junction x="71.12" y="-27.94"/>
 </segment>
 <segment>
@@
 <junction x="241.3" y="40.64"/>
 </segment>
+<segment>
+<pinref part="R11" gate="G$1" pin="1"/>
+<pinref part="U$16" gate="G$1" pin="GND"/>
+</segment>
 </net>
 <net name="I2SLRCK" class="0">
 <segment>
 <pinref part="U3" gate="G$1" pin="LRCK"/>
-<wire x1="127" y1="33.02" x2="124.46" y2="33.02" width="0.1524" layer="91"/>
 <label x="111.76" y="33.02" size="1.27" layer="95" rot="R180" xref="yes"/>
-<pinref part="RN1" gate="A" pin="1"/>
-<wire x1="124.46" y1="33.02" x2="114.3" y2="33.02" width="0.1524" layer="91"/>
-<wire x1="114.3" y1="33.02" x2="111.76" y2="33.02" width="0.1524" layer="91"/>
-<junction x="114.3" y="33.02"/>
-<pinref part="RN1" gate="A" pin="2"/>
-<junction x="124.46" y="33.02"/>
+<wire x1="127" y1="33.02" x2="111.76" y2="33.02" width="0.1524" layer="91"/>
 </segment>
 <segment>
@@
 <segment>
 <pinref part="U3" gate="G$1" pin="BICK"/>
-<wire x1="127" y1="30.48" x2="124.46" y2="30.48" width="0.1524" layer="91"/>
 <label x="111.76" y="30.48" size="1.27" layer="95" rot="R180" xref="yes"/>
-<pinref part="RN1" gate="C" pin="1"/>
-<wire x1="124.46" y1="30.48" x2="114.3" y2="30.48" width="0.1524" layer="91"/>
-<wire x1="114.3" y1="30.48" x2="111.76" y2="30.48" width="0.1524" layer="91"/>
-<junction x="114.3" y="30.48"/>
-<pinref part="RN1" gate="C" pin="2"/>
-<junction x="124.46" y="30.48"/>
+<wire x1="127" y1="30.48" x2="111.76" y2="30.48" width="0.1524" layer="91"/>
 </segment>
 <segment>
@@
 <segment>
 <pinref part="U3" gate="G$1" pin="SDTI"/>
-<wire x1="127" y1="27.94" x2="124.46" y2="27.94" width="0.1524" layer="91"/>
 <label x="111.76" y="27.94" size="1.27" layer="95" rot="R180" xref="yes"/>
-<pinref part="RN1" gate="B" pin="1"/>
-<wire x1="124.46" y1="27.94" x2="114.3" y2="27.94" width="0.1524" layer="91"/>
-<wire x1="114.3" y1="27.94" x2="111.76" y2="27.94" width="0.1524" layer="91"/>
-<junction x="114.3" y="27.94"/>
-<pinref part="RN1" gate="B" pin="2"/>
-<junction x="124.46" y="27.94"/>
+<wire x1="127" y1="27.94" x2="111.76" y2="27.94" width="0.1524" layer="91"/>
 </segment>
 <segment>
 <pinref part="U11" gate="G$1" pin="SOSCO/RPA4/T1CK/CTED9/PMA1/RA4"/>
 <wire x1="236.22" y1="-58.42" x2="261.62" y2="-58.42" width="0.1524" layer="91"/>
+<label x="261.62" y="-58.42" size="1.27" layer="95" xref="yes"/>
 </segment>
 </net>
@@
 <segment>
 <pinref part="U3" gate="G$1" pin="MCLK"/>
-<wire x1="127" y1="50.8" x2="124.46" y2="50.8" width="0.1524" layer="91"/>
 <label x="111.76" y="50.8" size="1.27" layer="95" rot="R180" xref="yes"/>
-<pinref part="RN1" gate="D" pin="1"/>
-<wire x1="124.46" y1="50.8" x2="114.3" y2="50.8" width="0.1524" layer="91"/>
-<wire x1="114.3" y1="50.8" x2="111.76" y2="50.8" width="0.1524" layer="91"/>
-<junction x="114.3" y="50.8"/>
-<pinref part="RN1" gate="D" pin="2"/>
-<junction x="124.46" y="50.8"/>
+<wire x1="127" y1="50.8" x2="111.76" y2="50.8" width="0.1524" layer="91"/>
 </segment>
 <segment>
 <pinref part="U11" gate="G$1" pin="VREF-/CVREF-/AN1/RPA1/CTED2/RA1"/>
 <wire x1="236.22" y1="-66.04" x2="261.62" y2="-66.04" width="0.1524" layer="91"/>
+<label x="261.62" y="-66.04" size="1.27" layer="95" xref="yes"/>
 </segment>
 </net>
@@
 </segment>
 <segment>
-<pinref part="U1" gate="G$1" pin="NC"/>
 <pinref part="+3V10" gate="G$1" pin="+3V3"/>
-<wire x1="22.86" y1="35.56" x2="27.94" y2="35.56" width="0.1524" layer="91"/>
 <pinref part="C11" gate="G$1" pin="1"/>
 <wire x1="27.94" y1="35.56" x2="30.48" y2="35.56" width="0.1524" layer="91"/>
-<junction x="27.94" y="35.56"/>
 </segment>
 <segment>
@@
 <pinref part="+3V17" gate="G$1" pin="+3V3"/>
 </segment>
+<segment>
+<pinref part="U1" gate="G$1" pin="VCC"/>
+<pinref part="+3V18" gate="G$1" pin="+3V3"/>
+</segment>
 </net>
 <net name="N$1" class="0">
@@
 <junction x="231.14" y="20.32"/>
 </segment>
+<segment>
+<pinref part="U11" gate="G$1" pin="AN11/RPB13/CTPLS/PMRD/RB13"/>
+<wire x1="101.6" y1="-63.5" x2="93.98" y2="-63.5" width="0.1524" layer="91"/>
+<label x="93.98" y="-63.5" size="1.27" layer="95" rot="R180" xref="yes"/>
+</segment>
 </net>
 <net name="MMCCD" class="0">
@@
 <label x="327.66" y="-50.8" size="1.27" layer="95" xref="yes"/>
 <pinref part="U12" gate="G$1" pin="3"/>
-</segment>
-</net>
-<net name="N$18" class="0">
-<segment>
-<pinref part="U11" gate="G$1" pin="AN11/RPB13/CTPLS/PMRD/RB13"/>
-<wire x1="101.6" y1="-63.5" x2="93.98" y2="-63.5" width="0.1524" layer="91"/>
-<label x="93.98" y="-63.5" size="1.27" layer="95" rot="R180" xref="yes"/>
 </segment>
 </net>
@@
 </segment>
 </net>
-<net name="N$26" class="0">
-<segment>
-<pinref part="U11" gate="G$1" pin="VREF+/CVREF+/AN0/C3INC/RPA0/CTED1/RA0"/>
-<wire x1="236.22" y1="-68.58" x2="248.92" y2="-68.58" width="0.1524" layer="91"/>
-</segment>
-</net>
 <net name="SDO" class="0">
 <segment>
@@
 </segment>
 </net>
-<net name="N$16" class="0">
+<net name="VSENSE" class="0">
 <segment>
 <pinref part="U11" gate="G$1" pin="AN12/PMD0/RB12"/>
 <wire x1="93.98" y1="-66.04" x2="101.6" y2="-66.04" width="0.1524" layer="91"/>
-</segment>
-</net>
+<label x="93.98" y="-66.04" size="1.27" layer="95" rot="R180" xref="yes"/>
+</segment>
+</net>
+<net name="BATS" class="0">
+<segment>
+<pinref part="R10" gate="G$1" pin="1"/>
+<pinref part="R11" gate="G$1" pin="2"/>
+<wire x1="71.12" y1="-38.1" x2="71.12" y2="-40.64" width="0.1524" layer="91"/>
+<wire x1="71.12" y1="-40.64" x2="66.04" y2="-40.64" width="0.1524" layer="91"/>
+<junction x="71.12" y="-40.64"/>
+<label x="66.04" y="-40.64" size="1.27" layer="95" rot="R180" xref="yes"/>
+</segment>
+<segment>
+<pinref part="U11" gate="G$1" pin="VREF+/CVREF+/AN0/C3INC/RPA0/CTED1/RA0"/>
+<wire x1="236.22" y1="-68.58" x2="261.62" y2="-68.58" width="0.1524" layer="91"/>
+<label x="261.62" y="-68.58" size="1.27" layer="95" xref="yes"/>
+</segment>
+</net>
